Commit message: add navigation and localisation

File: src/shesnar/urdf/lidar.xacro (robot description, xacro)
@@ -4,5 +4,5 @@
         <parent link="body"/>
         <child link="laser_frame"/>
-        <origin xyz="0 0 0.18" rpy="0 0 0"/>
+        <origin xyz="0 0 0.18" rpy="0 0 -2.085"/>
     </joint>
     <link name="laser_frame">

File: src/shesnar/urdf/robot_core.xacro (robot description, xacro)
@@ -15,9 +15,16 @@
         <origin xyz="0 0 0"/>
     </joint>
+    <link name="base_footprint"></link>
+    <joint name="base_footprint_joint" type="fixed">
+        <parent link="base_link"/>
+        <child link="base_footprint"/>
+        <origin xyz="0 0 0"/>
+    </joint>
     <link name="body">
         <visual>
             <origin xyz="-0.18 -0.1 0" rpy="0 0 0" />
             <geometry>
-                <mesh filename="package://shesnar/meshes/body.dae" scale="0.001 0.001 0.001"/>
+                <mesh filename="package://shesnar/meshes/body.dae" scale="0.001 0.001 0.001" rpy="0 0 1.04"/>
+            <!-- <cylinder radius="0.20" length="0.12"/> -->
             </geometry>
             <material name="">
